File: Hardware/SparkFun_MicroMod_GNSS_Function_Board_ZED-F9P.sch (EAGLE design)
At the start: 107 parts, among them J1 USB Female Type C Connector, J10 U.FL, J11 455-1750-1-ND, J15 QWIIC_VERT, J16 QWIIC_RA, J18 Bus Selection, J2 MICROMOD_STANDARD, J3 Bus Selection, Q1 DMP21D0UT-7, U1 SN74LVC1G66DRYR, U10 SN74AUP1T04, U11 SN74AUP1T04, U2 3.3V, U3 EEPROM, U4 74LVC4066D_QUAD_BILATERAL_SWI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, U5 74LVC4066D_QUAD_BILATERAL_SWI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, U6 OPA344, U7 74LVC541A, U8 U-BLOX_ZED-F9P, U9 FIN1017MX

Commit message: Renamed for release. Some updates post DR.
Parts:
- removed J15: QWIIC_VERT, SparkFun-Connectors:QWIIC_CONNECTOR
- removed J16: QWIIC_RA, SparkFun-Connectors:QWIIC_CONNECTORJS-1MM
- removed TP1, TP15, TP16, TP17, TP18, TP19, TP2, TP3, TP4: TEST-POINT3, SparkFun-Connectors:TEST-POINT3
- added R18: 10k, SparkFun-Resistors:10KOHM-0603-1/10W-1%
- D6: value BLUE -> YELLOW; device SparkFun-LED:LED-BLUE0603 -> SparkFun-LED:LED-YELLOW0603
- J2: value MICROMOD_STANDARD -> MICROMOD_FUNCTION_STANDARD; device SparkFun-MicroMod-Function:MICROMOD_STANDARD -> SparkFun-MicroMod:MICROMOD_FUNCTION_STANDARD
Connections:
- net !RESET!: no longer TP18.1
- net 3.3V: no longer J15.2, J16.2
- net 5V: now also R18.1
- net EXTINT: no longer TP19.1
- net GND: no longer J15.1, J16.1, TP2.1
- net GND_RF: no longer TP4.1
- net MM_SCL: no longer J15.4, J16.4
- net MM_SDA: no longer J15.3, J16.3
- net PWR_EN: now also R18.2
- net RX2/RTCM: no longer TP15.1
- net TX2/RTCM: no longer TP16.1
- net V_BATT: no longer TP3.1
- net V_ZED: no longer TP1.1
- net ZED_!SAFEBOOT!: no longer TP17.1
Other:
- note removed: "Qwiic Connector"
- moved on the sheet: C14, C15, C16, J11, J12, J14, J17, J18, J5, J6, J8, J9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

Commit message: Add part, update lib, resize sch parts, bulk brd update.
Add NLAST SPST switch.
Update POCI/PICO.
Make all resistors possible 0402. (Only 10ohm and 68.1k res are still 0603)
Parts:
- removed J18, J3: Bus Selection, SparkFun-Connectors:CONN_03LOCK
- added JP7, JP8: JUMPER-SMT_3_1-NC_TRACE_SILK, SparkFun-Jumpers:JUMPER-SMT_3_1-NC_TRACE_SILK
- C8: device MicroMod_Function_GNSS_ublox_ZED_F9P:CBR04C470J5GAC -> SparkFun_MicroMod_GNSS_Function_Board_ZED-F9P:CBR04C470J5GAC
- J11: device SparkFun-Connectors:CONN_03 -> SparkFun-Connectors:CONN_031X03_NO_SILK
- J12, J4, J5, J6, J8, J9: device SparkFun-Connectors:CONN_01 -> SparkFun-Connectors:CONN_01PTH_NO_SILK_YES_STOP
- J13, J14: device SparkFun-Connectors:CONN_02 -> SparkFun-Connectors:CONN_021X02_NO_SILK
- J17: device SparkFun-Connectors:CONN_04PTH -> SparkFun-Connectors:CONN_041X04_NO_SILK
- L1: device MicroMod_Function_GNSS_ublox_ZED_F9P:LQW15AWR15J80D -> SparkFun_MicroMod_GNSS_Function_Board_ZED-F9P:LQW15AWR15J80D
- Q1: device MicroMod_Function_GNSS_ublox_ZED_F9P:DMP21D0UT-7 -> SparkFun_MicroMod_GNSS_Function_Board_ZED-F9P:DMP21D0UT-7
- R1, R10, R11, R17, R18: device SparkFun-Resistors:10KOHM-0603-1/10W-1% -> SparkFun-Resistors:10KOHM-0402-1/16W-1%
- R12, R8, R9: value 1k -> 1KOHM-0402-1/16W-1%; device SparkFun-Resistors:1KOHM-0603-1/10W-1% -> SparkFun-Resistors:1KOHM-0402-1/16W-1%
- R13, R16: value 100k -> 100K; device SparkFun-Resistors:100KOHM-0603-1/10W-1% -> SparkFun-Resistors:100KOHM-0402-1/16W-1%
- R2, R3: device SparkFun-Resistors:5.1KOHM5.1KOHM-0603-1/10W-1% -> SparkFun-Resistors:5.1KOHM-0402-1/16W-1%
- R4: value 3.3k -> 3.3K; device SparkFun-Resistors:3.3KOHM-0603-1/10W-1% -> SparkFun-Resistors:3.3KOHM-0402T-1/16W-1%; RES (none) -> 3.3k
- R7: value 1k -> 1KOHM-0402-1/16W-1%; device SparkFun-Resistors:1KOHM-0603-1/10W-1% -> SparkFun-Resistors:1KOHM-0402-1/16W-1%; RES (none) -> 1k
- U1: value SN74LVC1G66DRYR -> NLAST4501DFT2G; device MicroMod_Function_GNSS_ublox_ZED_F9P:SN74LVC1G66DRYR -> SparkFun_MicroMod_GNSS_Function_Board_ZED-F9P:NLAST4501DFT2G
- U10, U11: device MicroMod_Function_GNSS_ublox_ZED_F9P:SN74AUP1T04DCK -> SparkFun_MicroMod_GNSS_Function_Board_ZED-F9P:SN74AUP1T04DCK
- U7: device MicroMod_Function_GNSS_ublox_ZED_F9P:74LVC541ABQ -> SparkFun_MicroMod_GNSS_Function_Board_ZED-F9P:74LVC541ABQ
- U8: device MicroMod_Function_GNSS_ublox_ZED_F9P:U-BLOX_ZED-F9P -> SparkFun_MicroMod_GNSS_Function_Board_ZED-F9P:U-BLOX_ZED-F9P
- U9: device MicroMod_Function_GNSS_ublox_ZED_F9P:FIN1017MX -> SparkFun_MicroMod_GNSS_Function_Board_ZED-F9P:FIN1017MX
Connections:
- net MM_CIPO renamed MM_POCI
- net MM_COPI renamed MM_PICO
- removed net N$10: J18.1, R17.1
- removed net N$11: J3.1, R10.1
- removed net N$12: J3.3, R11.2
- removed net ZED_RX/COPI: U4.4Y, U5.4Y, U8.RX/COPI
- removed net ZED_TX/CIPO: U4.3Y, U5.3Y, U8.TX/CIPO
- new net N$1: JP7.1, R10.1
- new net N$2: JP7.3, R11.2
- new net N$5: JP8.3, R17.1
- new net ZED_RX/PICO: U4.4Y, U5.4Y, U8.RX/PICO
- new net ZED_TX/POCI: U4.3Y, U5.3Y, U8.TX/POCI
- net GND_RF: now also JP8.1, U1.GND; no longer J18.3, U1.VSS
- net V_USB: now also U1.COM, U1.VCC; no longer U1.A_IN
- net V_ZED: now also U1.EN; no longer U1.CTRL_IN, U1.VCC
- net ZED_ANT_OFF: now also JP7.2; no longer J3.2
- net ZED_DSEL: now also JP8.2; no longer J18.2
- net ZED_USB_DET: now also U1.NO; no longer U1.A_OUT
Other:
- note added: "Cut jumper and solder 1-2 when using antenna supervisor."
- note added: "To use SPI cut jumper and connect side labeled "SPI"."
- note removed: "Move jumper to 1-2 when using antenna supervisor."
- note removed: "To use SPI simply move the 2-pin jumper to the side labeled "SPI"."
- moved on the sheet: R10, R11, R17

Commit message: Completed updates post DR.
Change PPS LED to Yellow.
U1 make power V_USB, not V_ZED.
Add PUR on PWR_EN.
Remove TPs where PTH exists.
Remove Qwiic connectors.
Change U1 to be a bigger package.
Change CIPO/COPI to PICO/POCI.
Route out from center of pad.
Remove silk from PTHs.
Fix skinny VIN trace.
Change 0.2mm vias to 0.3mm vias.
Change 0.35mm vias to 0.3mm vias where possible.
Set layers correctly on board so 2 and 15 are in correct location.
Reset Grid for design.
Change VZ LED silk to PWR.
Change Silk description.
Change i2c silk to have superscript 2.
Change CIPO/COPI to PICO/POCI.
Change version number to v01.
DRC Wire Stubs.
GND pour between power traces on L15.
GND pour between SPI/UART traces on L2.
Acid traps.
Change SS jumpers to SMD jumpers.
Board Dimensions change.
Space out capacitors on board.
Cover ANT with Solder Mask.
Remove copper on L1 from under U.FL.
Write Silk for L1/L2 antenna.
Remove TP silk.
WP Jumper label needs to be rounded on end.
Change names everywhere to SparkFun MicroMod GNSS Function Board - ZED-F9P.
Move U1 origin to center of device.
Remove $ from new FPs.
Text ratio for tDocu.
Changed all passives to 0402 except 10 ohm and 68.1kohm Res.
Parts:
- JP3: value JUMPER-SMT_2_NC_TRACE_SILK -> JUMPER-SMT_2_NO_SILK; device SparkFun-Jumpers:JUMPER-SMT_2_NC_TRACE_SILK -> SparkFun-Jumpers:JUMPER-SMT_2_NO_SILK
- R12, R7: value 1KOHM-0402-1/16W-1% -> 100k; device SparkFun-Resistors:1KOHM-0402-1/16W-1% -> SparkFun-Resistors:100KOHM-0402T-1/16W-1%
- R13, R16: value 100K -> 100k; device SparkFun-Resistors:100KOHM-0402-1/16W-1% -> SparkFun-Resistors:100KOHM-0402T-1/16W-1%
- R2, R3: device SparkFun-Resistors:5.1KOHM-0402-1/16W-1% -> SparkFun-Resistors:5.1KOHM-0402T-1/16W-1%
Changed lines of the file:
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@@
 <layers>
 <layer number="1" name="Top" color="4" fill="1" visible="no" active="no"/>
-<layer number="2" name="Route2" color="1" fill="3" visible="no" active="no"/>
+<layer number="2" name="Route2" color="13" fill="3" visible="no" active="no"/>
 <layer number="3" name="Route3" color="4" fill="3" visible="no" active="no"/>
 <layer number="4" name="Route4" color="1" fill="4" visible="no" active="no"/>
@@
 <layer number="13" name="Route13" color="4" fill="5" visible="no" active="no"/>
 <layer number="14" name="Route14" color="1" fill="6" visible="no" active="no"/>
-<layer number="15" name="Route15" color="4" fill="6" visible="no" active="no"/>
-<layer number="16" name="Bottom" color="1" fill="1" visible="no" active="no"/>
+<layer number="15" name="Route15" color="47" fill="6" visible="no" active="no"/>
+<layer number="16" name="Bottom" color="9" fill="1" visible="no" active="no"/>
 <layer number="17" name="Pads" color="2" fill="1" visible="no" active="no"/>
 <layer number="18" name="Vias" color="2" fill="1" visible="no" active="no"/>
@@
 <part name="SUPPLY2" library="SparkFun-PowerSymbols" deviceset="3.3V" device=""/>
 <part name="GND2" library="SparkFun-PowerSymbols" deviceset="GND" device=""/>
-<part name="R2" library="SparkFun-Resistors" deviceset="5.1KOHM" device="-0402-1/16W-1%" value="5.1k"/>
-<part name="R3" library="SparkFun-Resistors" deviceset="5.1KOHM" device="-0402-1/16W-1%" value="5.1k"/>
+<part name="R2" library="SparkFun-Resistors" deviceset="5.1KOHM" device="-0402T-1/16W-1%" value="5.1k"/>
+<part name="R3" library="SparkFun-Resistors" deviceset="5.1KOHM" device="-0402T-1/16W-1%" value="5.1k"/>
 <part name="SUPPLY4" library="SparkFun-PowerSymbols" deviceset="V_USB" device=""/>
 <part name="SUPPLY5" library="SparkFun-PowerSymbols" deviceset="V_USB" device=""/>
@@
 <part name="SUPPLY25" library="SparkFun-PowerSymbols" deviceset="VIN" device=""/>
 <part name="D1" library="SparkFun-DiscreteSemi" deviceset="DIODE-SCHOTTKY" device="-BAT60A" value="3A/10V/280mV"/>
-<part name="R7" library="SparkFun-Resistors" deviceset="1KOHM" device="-0402-1/16W-1%" value="1KOHM-0402-1/16W-1%">
+<part name="R7" library="SparkFun-Resistors" deviceset="100KOHM" device="-0402T-1/16W-1%" value="100k">
 <attribute name="RES" value="1k"/>
 </part>
@@
 <part name="SUPPLY7" library="SparkFun-PowerSymbols" deviceset="V_BATT" device=""/>
 <part name="SUPPLY19" library="SparkFun-PowerSymbols" deviceset="VDD" device="" value="V_ZED"/>
-<part name="R16" library="SparkFun-Resistors" deviceset="100KOHM" device="-0402-1/16W-1%" value="100K"/>
+<part name="R16" library="SparkFun-Resistors" deviceset="100KOHM" device="-0402T-1/16W-1%" value="100k"/>
 <part name="U8" library="SparkFun_MicroMod_GNSS_Function_Board_ZED-F9P" deviceset="U-BLOX_ZED-F9P" device=""/>
 <part name="C10" library="SparkFun-Capacitors" deviceset="0.1UF" device="-0402T-16V-10%" value="0.1uF"/>
@@
 <part name="C5" library="SparkFun-Capacitors" deviceset="10NF" device="-0402T-25V-10%-X7R-WE" value="10nF"/>
 <part name="U$2" library="SparkFun_MicroMod_GNSS_Function_Board_ZED-F9P" deviceset="GND_RF" device=""/>
-<part name="R13" library="SparkFun-Resistors" deviceset="100KOHM" device="-0402-1/16W-1%" value="100K"/>
+<part name="R13" library="SparkFun-Resistors" deviceset="100KOHM" device="-0402T-1/16W-1%" value="100k"/>
 <part name="Q1" library="SparkFun_MicroMod_GNSS_Function_Board_ZED-F9P" deviceset="DMP21D0UT" device="-7" value="DMP21D0UT-7"/>
 <part name="U$8" library="SparkFun_MicroMod_GNSS_Function_Board_ZED-F9P" deviceset="V_RF" device=""/>
@@
 <part name="SUPPLY28" library="SparkFun-PowerSymbols" deviceset="3.3V" device=""/>
 <part name="SUPPLY29" library="SparkFun-PowerSymbols" deviceset="3.3V" device=""/>
-<part name="JP3" library="SparkFun-Jumpers" deviceset="JUMPER-SMT_2_NC_TRACE" device="_SILK" package3d_urn="urn:adsk.eagle:package:39281/1"/>
+<part name="JP3" library="SparkFun-Jumpers" deviceset="JUMPER-SMT_2_NO" device="_SILK" package3d_urn="urn:adsk.eagle:package:39279/1"/>
 <part name="GND5" library="SparkFun-PowerSymbols" deviceset="GND" device=""/>
 <part name="JP1" library="SparkFun-Jumpers" deviceset="JUMPER-SMT_2_NO" device="_SILK" package3d_urn="urn:adsk.eagle:package:39279/1"/>
@@
 <part name="C15" library="SparkFun-Capacitors" deviceset="0.1UF" device="-0402T-16V-10%" value="0.1uF"/>
 <part name="C16" library="SparkFun-Capacitors" deviceset="0.1UF" device="-0402T-16V-10%" value="0.1uF"/>
-<part name="R12" library="SparkFun-Resistors" deviceset="1KOHM" device="-0402-1/16W-1%" value="1KOHM-0402-1/16W-1%">
+<part name="R12" library="SparkFun-Resistors" deviceset="100KOHM" device="-0402T-1/16W-1%" value="100k">
 <attribute name="RESISTANCE" value="1k"/>
 </part>

Commit message: update to v02 for mfgr error.
Other:
- note added: "v02"
- note removed: "v01"
Changed lines of the file:
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@@
 <grid distance="0.1" unitdist="inch" unit="inch" style="lines" multiple="1" display="no" altdistance="0.01" altunitdist="inch" altunit="inch"/>
 <layers>
-<layer number="1" name="Top" color="4" fill="1" visible="yes" active="no"/>
-<layer number="2" name="Route2" color="13" fill="3" visible="yes" active="no"/>
-<layer number="3" name="Route3" color="4" fill="3" visible="yes" active="no"/>
-<layer number="4" name="Route4" color="1" fill="4" visible="yes" active="no"/>
-<layer number="5" name="Route5" color="4" fill="4" visible="yes" active="no"/>
-<layer number="6" name="Route6" color="1" fill="8" visible="yes" active="no"/>
-<layer number="7" name="Route7" color="4" fill="8" visible="yes" active="no"/>
-<layer number="8" name="Route8" color="1" fill="2" visible="yes" active="no"/>
-<layer number="9" name="Route9" color="4" fill="2" visible="yes" active="no"/>
-<layer number="10" name="Route10" color="1" fill="7" visible="yes" active="no"/>
-<layer number="11" name="Route11" color="4" fill="7" visible="yes" active="no"/>
-<layer number="12" name="Route12" color="1" fill="5" visible="yes" active="no"/>
-<layer number="13" name="Route13" color="4" fill="5" visible="yes" active="no"/>
-<layer number="14" name="Route14" color="1" fill="6" visible="yes" active="no"/>
-<layer number="15" name="Route15" color="47" fill="6" visible="yes" active="no"/>
-<layer number="16" name="Bottom" color="9" fill="1" visible="yes" active="no"/>
-<layer number="17" name="Pads" color="2" fill="1" visible="yes" active="no"/>
-<layer number="18" name="Vias" color="2" fill="1" visible="yes" active="no"/>
-<layer number="19" name="Unrouted" color="6" fill="1" visible="yes" active="no"/>
-<layer number="20" name="Dimension" color="24" fill="1" visible="yes" active="no"/>
-<layer number="21" name="tPlace" color="16" fill="1" visible="yes" active="no"/>
-<layer number="22" name="bPlace" color="14" fill="1" visible="yes" active="no"/>
-<layer number="23" name="tOrigins" color="15" fill="1" visible="yes" active="no"/>
-<layer number="24" name="bOrigins" color="15" fill="1" visible="yes" active="no"/>
-<layer number="25" name="tNames" color="7" fill="1" visible="yes" active="no"/>
-<layer number="26" name="bNames" color="7" fill="1" visible="yes" active="no"/>
-<layer number="27" name="tValues" color="7" fill="1" visible="yes" active="no"/>
-<layer number="28" name="bValues" color="7" fill="1" visible="yes" active="no"/>
+<layer number="1" name="Top" color="4" fill="1" visible="no" active="no"/>
+<layer number="2" name="Route2" color="13" fill="3" visible="no" active="no"/>
+<layer number="3" name="Route3" color="4" fill="3" visible="no" active="no"/>
+<layer number="4" name="Route4" color="1" fill="4" visible="no" active="no"/>
+<layer number="5" name="Route5" color="4" fill="4" visible="no" active="no"/>
+<layer number="6" name="Route6" color="1" fill="8" visible="no" active="no"/>
+<layer number="7" name="Route7" color="4" fill="8" visible="no" active="no"/>
+<layer number="8" name="Route8" color="1" fill="2" visible="no" active="no"/>
+<layer number="9" name="Route9" color="4" fill="2" visible="no" active="no"/>
+<layer number="10" name="Route10" color="1" fill="7" visible="no" active="no"/>
+<layer number="11" name="Route11" color="4" fill="7" visible="no" active="no"/>
+<layer number="12" name="Route12" color="1" fill="5" visible="no" active="no"/>
+<layer number="13" name="Route13" color="4" fill="5" visible="no" active="no"/>
+<layer number="14" name="Route14" color="1" fill="6" visible="no" active="no"/>
+<layer number="15" name="Route15" color="47" fill="6" visible="no" active="no"/>
+<layer number="16" name="Bottom" color="9" fill="1" visible="no" active="no"/>
+<layer number="17" name="Pads" color="2" fill="1" visible="no" active="no"/>
+<layer number="18" name="Vias" color="2" fill="1" visible="no" active="no"/>
+<layer number="19" name="Unrouted" color="6" fill="1" visible="no" active="no"/>
+<layer number="20" name="Dimension" color="24" fill="1" visible="no" active="no"/>
+<layer number="21" name="tPlace" color="16" fill="1" visible="no" active="no"/>
+<layer number="22" name="bPlace" color="14" fill="1" visible="no" active="no"/>
+<layer number="23" name="tOrigins" color="15" fill="1" visible="no" active="no"/>
+<layer number="24" name="bOrigins" color="15" fill="1" visible="no" active="no"/>
+<layer number="25" name="tNames" color="7" fill="1" visible="no" active="no"/>
+<layer number="26" name="bNames" color="7" fill="1" visible="no" active="no"/>
+<layer number="27" name="tValues" color="7" fill="1" visible="no" active="no"/>
+<layer number="28" name="bValues" color="7" fill="1" visible="no" active="no"/>
 <layer number="29" name="tStop" color="7" fill="3" visible="no" active="no"/>
 <layer number="30" name="bStop" color="7" fill="6" visible="no" active="no"/>
@@
 <layer number="35" name="tGlue" color="7" fill="4" visible="no" active="no"/>
 <layer number="36" name="bGlue" color="7" fill="5" visible="no" active="no"/>
-<layer number="37" name="tTest" color="7" fill="1" visible="yes" active="no"/>
-<layer number="38" name="bTest" color="7" fill="1" visible="yes" active="no"/>
+<layer number="37" name="tTest" color="7" fill="1" visible="no" active="no"/>
+<layer number="38" name="bTest" color="7" fill="1" visible="no" active="no"/>
 <layer number="39" name="tKeepout" color="4" fill="11" visible="no" active="no"/>
 <layer number="40" name="bKeepout" color="1" fill="11" visible="no" active="no"/>
@@
 <layer number="44" name="Drills" color="7" fill="1" visible="no" active="no"/>
 <layer number="45" name="Holes" color="7" fill="1" visible="no" active="no"/>
-<layer number="46" name="Milling" color="3" fill="1" visible="yes" active="no"/>
-<layer number="47" name="Measures" color="7" fill="1" visible="yes" active="no"/>
-<layer number="48" name="Document" color="7" fill="1" visible="yes" active="no"/>
-<layer number="49" name="Reference" color="7" fill="1" visible="yes" active="no"/>
-<layer number="50" name="dxf" color="7" fill="1" visible="yes" active="no"/>
-<layer number="51" name="tDocu" color="6" fill="1" visible="yes" active="no"/>
-<layer number="52" name="bDocu" color="7" fill="1" visible="yes" active="no"/>
-<layer number="53" name="tGND_GNDA" color="7" fill="9" visible="yes" active="no"/>
-<layer number="54" name="bGND_GNDA" color="1" fill="9" visible="yes" active="no"/>
-<layer number="56" name="wert" color="7" fill="1" visible="yes" active="no"/>
-<layer number="57" name="tCAD" color="7" fill="1" visible="yes" active="no"/>
-<layer number="58" name="bCAD" color="7" fill="1" visible="yes" active="no"/>
-<layer number="59" name="tCarbon" color="7" fill="1" visible="yes" active="no"/>
-<layer number="60" name="bCarbon" color="7" fill="1" visible="yes" active="no"/>
+<layer number="46" name="Milling" color="3" fill="1" visible="no" active="no"/>
+<layer number="47" name="Measures" color="7" fill="1" visible="no" active="no"/>
+<layer number="48" name="Document" color="7" fill="1" visible="no" active="no"/>
+<layer number="49" name="Reference" color="7" fill="1" visible="no" active="no"/>
+<layer number="50" name="dxf" color="7" fill="1" visible="no" active="no"/>
+<layer number="51" name="tDocu" color="6" fill="1" visible="no" active="no"/>
+<layer number="52" name="bDocu" color="7" fill="1" visible="no" active="no"/>
+<layer number="53" name="tGND_GNDA" color="7" fill="9" visible="no" active="no"/>
+<layer number="54" name="bGND_GNDA" color="1" fill="9" visible="no" active="no"/>
+<layer number="56" name="wert" color="7" fill="1" visible="no" active="no"/>
+<layer number="57" name="tCAD" color="7" fill="1" visible="no" active="no"/>
+<layer number="58" name="bCAD" color="7" fill="1" visible="no" active="no"/>
+<layer number="59" name="tCarbon" color="7" fill="1" visible="no" active="no"/>
+<layer number="60" name="bCarbon" color="7" fill="1" visible="no" active="no"/>
 <layer number="88" name="SimResults" color="9" fill="1" visible="yes" active="yes"/>
 <layer number="89" name="SimProbes" color="9" fill="1" visible="yes" active="yes"/>
@@
 <text x="96.774" y="86.106" size="2.54" layer="94" font="vector" align="center">MicroMod Function Connector</text>
 <text x="348.234" y="11.176" size="2.54" layer="94" font="vector">A. Brudner</text>
-<text x="421.894" y="6.096" size="2.54" layer="94" font="vector">v01</text>
+<text x="421.894" y="6.096" size="2.54" layer="94" font="vector">v02</text>
 <text x="71.12" y="269.24" size="2.54" layer="94" font="vector" align="center">ZED-F9P USB (u-center)</text>
 <text x="111.76" y="203.2" size="2.54" layer="94" font="vector" align="center">ZED-F9P Backup Battery</text>
