File: Hardware/SparkFun_MicroMod_GNSS_Function_Board_ZED-F9P.sch (EAGLE design)
At the start: 97 parts, among them J1 USB Female Type C Connector, J10 U.FL, J11 455-1750-1-ND, J2 MICROMOD_FUNCTION_STANDARD, Q1 DMP21D0UT-7, U1 NLAST4501DFT2G, U10 SN74AUP1T04, U11 SN74AUP1T04, U2 3.3V, U3 EEPROM, U4 74LVC4066D_QUAD_BILATERAL_SWI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, U5 74LVC4066D_QUAD_BILATERAL_SWI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, U6 OPA344, U7 74LVC541A, U8 U-BLOX_ZED-F9P, U9 FIN1017MX

Commit message: v03 protos update.
Center and update flags.
Fix RTK STAT circuit.
Fix voltage divider for USB detect.
Add I2C PURs.
Add a PUR for the reset line outside isolation.
Changed PWR LED resistor to 1k.
Moved PPS and RTK LEDs to top of board.
Removed RF_GND.
Rerouted board.
Parts:
- removed J17: (no value), SparkFun-Connectors:CONN_041X04_NO_SILK
- removed SUPPLYTIE1: 2PT_GND_TIE, SparkFun-PowerSymbols:2PT_GND_TIE
- added J3: (no value), SparkFun-Connectors:CONN_01PTH_NO_SILK_YES_STOP
- added JP9: JUMPER-SMT_3_1-NC_TRACE_SILK, SparkFun-Jumpers:JUMPER-SMT_3_1-NC_TRACE_SILK
- added R19: 47k, SparkFun-Resistors:47KOHM-0402-1/10W-1%
- added R20, R21: 10k, SparkFun-Resistors:10KOHM-0402T-1/16W-1%
- D4: value 0.5A/40V/420mV -> RED; device SparkFun-DiscreteSemi:DIODE-SCHOTTKY-PMEG4005EJ -> SparkFun-LED:LED-RED0603
- D5: value RED -> BLUE; device SparkFun-LED:LED-RED0603 -> SparkFun-LED:LED-BLUE0603
- D7: value BLUE -> 0.5A/40V/420mV; device SparkFun-LED:LED-BLUE0603 -> SparkFun-DiscreteSemi:DIODE-SCHOTTKY-PMEG4005EJ
- J10: value U.FL -> 455-1750-1-ND; device SparkFun-Connectors:U.FL2PIN -> SparkFun-Connectors:CONN_031X03_NO_SILK
- J11: value 455-1750-1-ND -> (none); device SparkFun-Connectors:CONN_031X03_NO_SILK -> SparkFun-Connectors:CONN_01PTH_NO_SILK_YES_STOP
- J12: device SparkFun-Connectors:CONN_01PTH_NO_SILK_YES_STOP -> SparkFun-Connectors:CONN_021X02_NO_SILK
- J14: device SparkFun-Connectors:CONN_021X02_NO_SILK -> SparkFun-Connectors:CONN_041X04_NO_SILK
- J6: device SparkFun-Connectors:CONN_01PTH_NO_SILK_YES_STOP -> SparkFun-Connectors:CONN_01PTH_NO_SILK_SMALL
- J7: device SparkFun-Connectors:CONN_01PTH_NO_SILK_SMALL -> SparkFun-Connectors:CONN_01PTH_NO_SILK_YES_STOP
- J9: value (none) -> U.FL; device SparkFun-Connectors:CONN_01PTH_NO_SILK_YES_STOP -> SparkFun-Connectors:U.FL2PIN
- JP7: value JUMPER-SMT_3_1-NC_TRACE_SILK -> JUMPER-SMT_3_2-NC_TRACE_SILK; device SparkFun-Jumpers:JUMPER-SMT_3_1-NC_TRACE_SILK -> SparkFun-Jumpers:JUMPER-SMT_3_2-NC_TRACE_SILK
- R1: device SparkFun-Resistors:10KOHM-0402-1/16W-1% -> SparkFun-Resistors:10KOHM-0402T-1/16W-1%
- R10: value 10k -> 27; device SparkFun-Resistors:10KOHM-0402-1/16W-1% -> SparkFun-Resistors:27OHM
- R11: value 10k -> 2.2k; device SparkFun-Resistors:10KOHM-0402-1/16W-1% -> SparkFun-Resistors:2.2KOHM-0402T-1/16W-1%
- R12: value 100k -> 2.2k; device SparkFun-Resistors:100KOHM-0402T-1/16W-1% -> SparkFun-Resistors:2.2KOHM-0402T-1/16W-1%; RESISTANCE 1k -> (none)
- R13: value 100k -> 10k; device SparkFun-Resistors:100KOHM-0402T-1/16W-1% -> SparkFun-Resistors:10KOHM-0402T-1/16W-1%
- R14: value 10 -> 10k; device SparkFun-Resistors:10OHM-0603-1/10W-1% -> SparkFun-Resistors:10KOHM-0402T-1/16W-1%
- R15: value 68.1k -> 1k; device SparkFun-Resistors:68.1KOHM-0603-1/10W-1% -> SparkFun-Resistors:1KOHM-0402T-1/16W-1%; RESISTANCE (none) -> 1k
- R17: value 10k -> 10; device SparkFun-Resistors:10KOHM-0402-1/16W-1% -> SparkFun-Resistors:10OHM-0603-1/10W-1%
- R18: value 10k -> 22k; device SparkFun-Resistors:10KOHM-0402-1/16W-1% -> SparkFun-Resistors:22KOHM-0402_TIGHT-1/10W-1%
- R2: value 5.1k -> 10k; device SparkFun-Resistors:5.1KOHM-0402T-1/16W-1% -> SparkFun-Resistors:10KOHM-0402T-1/16W-1%
- R4: value 3.3K -> 5.1k; device SparkFun-Resistors:3.3KOHM-0402T-1/16W-1% -> SparkFun-Resistors:5.1KOHM-0402T-1/16W-1%; RES 3.3k -> (none)
- R5: value 27 -> 3.3K; device SparkFun-Resistors:27OHM -> SparkFun-Resistors:3.3KOHM-0402T-1/16W-1%; RES (none) -> 3.3k
- R6: value 27 -> 1k; device SparkFun-Resistors:27OHM -> SparkFun-Resistors:1KOHM-0402T-1/16W-1%
- R7: value 100k -> 1k; device SparkFun-Resistors:100KOHM-0402T-1/16W-1% -> SparkFun-Resistors:1KOHM-0402T-1/16W-1%; RES 1k -> (none)
- R8: value 1KOHM-0402-1/16W-1% -> 1k; device SparkFun-Resistors:1KOHM-0402-1/16W-1% -> SparkFun-Resistors:1KOHM-0402T-1/16W-1%
- R9: value 1KOHM-0402-1/16W-1% -> 27; device SparkFun-Resistors:1KOHM-0402-1/16W-1% -> SparkFun-Resistors:27OHM
Connections:
- removed net GND_RF: C10.2, C11.2, C12.2, C13.2, C15.2, C16.2, C4.2, C5.2, C6.2, C7.2, C9.2, D8.2, J10.GND, J8.1, J9.1, JP4.2, JP8.1, R11.1, R13.1, R16.1, SUPPLYTIE1.P$1, U1.GND, U10.GND, U11.GND, U4.GND, U5.GND, U6G2.P$V-, U7.GND, U8.GND
- removed net N$29 (its old number): D7.C, R9.2
- new net N$2: JP8.3, R14.2
- new net N$30: D4.C, R6.2
- new net N$9: JP7.1, R12.2
- net !RESET!: now also J12.1, R20.2; no longer J13.1
- net 3.3V: now also D7.A; no longer D4.A
- net 5V: now also R2.1; no longer R18.1
- net EXTINT: now also J13.1; no longer J14.1
- net GND: now also C10.2, C11.2, C12.2, C13.2, C15.2, C16.2, C4.2, C5.2, C6.2, C7.2, C9.2, D8.2, J10.3, J12.2, J14.1, J14.4, J4.1, J7.1, J8.1, J9.GND, JP4.2, JP9.1, R14.1, R16.1, R19.1, R4.1, U1.GND, U10.GND, U11.GND, U4.GND, U5.GND, U6G2.P$V-, U7.GND, U8.GND; no longer J11.3, J14.2, J17.1, J17.4, J6.1, JP5.1, R2.1, SUPPLYTIE1.P$2
- net MM_SCL: now also R11.1
- net MM_SDA: now also R12.1
- net N$1: now also JP8.1, R13.1; no longer JP7.1, R10.1
- net N$13: now also R15.1, R17.1; no longer R12.1, R14.1
- net N$14: now also R18.2, R19.2; no longer R15.2, R16.2
- net N$26: now also R6.1; no longer R7.1
- net N$27: now also JP6.2; no longer JP5.2
- net N$3: now also R3.2; no longer R2.2
- net N$32: now also D7.C, R5.2; no longer D4.C, R4.2
- net N$4: now also R4.2; no longer R3.2
- net N$48: now also R15.2, R16.2; no longer R12.2, R13.2
- net N$5: now also JP9.3, R21.1; no longer JP8.3, R17.1
- net N$7: now also J9.SIGNAL; no longer J10.SIGNAL
- net N$8: now also JP5.2, R7.1; no longer JP6.2, R9.1
- net PPS: no longer D6.A
- net PPS_DIFF_N: now also J14.3; no longer J17.3
- net PPS_DIFF_P: now also J14.2; no longer J17.2
- net PWR_EN: now also R2.2; no longer R18.2
- net RTK_STAT: no longer D7.A
- net RX2/RTCM: now also J10.1; no longer J11.1
- net TX2/RTCM: now also J10.2; no longer J11.2
- net USB_N: now also R10.1; no longer R6.1
- net USB_P: now also R9.1; no longer R5.1
- net V_BATT: now also J6.1, R5.1; no longer J7.1, R4.1
- net V_RF: now also R13.2; no longer R10.2
- net V_ZED: now also D4.A, J3.1, JP7.2, R20.1, R21.2; no longer J4.1, R17.2
- net ZED_!SAFEBOOT!: now also J11.1; no longer J12.1
- net ZED_ANT_!SHORT!: now also R17.2; no longer R14.2
- net ZED_ANT_OFF: now also JP8.2; no longer JP7.2
- net ZED_DSEL: now also JP9.2; no longer JP8.2
- net ZED_PPS: now also D6.A
- net ZED_RTK_STAT: now also JP5.1
- net ZED_USB_DET: now also R18.1; no longer R15.1
- net ZED_USB_N: now also R10.2; no longer R6.2
- net ZED_USB_P: now also R9.2; no longer R5.2
Other:
- note added: "Cut traces to remove pull-up resistors."
- note added: "RTK Solution: Off: None Blinking: Float On: Fixed"
- note added: "v03"
- note removed: "v02"
- moved on the sheet: C2, D5, D6, J13, J2, J4, J5, J6, J7, J8, JP2, JP4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
