File: Hardware/SparkFun_MicroMod_GNSS_Function_Board_ZED-F9P.sch (EAGLE design)
At the start: 100 parts, among them J1 USB Female Type C Connector, J10 455-1750-1-ND, J2 MICROMOD_FUNCTION_STANDARD, J9 U.FL, Q1 DMP21D0UT-7, U1 NLAST4501DFT2G, U10 SN74AUP1T04, U11 SN74AUP1T04, U2 3.3V, U3 EEPROM, U4 74LVC4066D_QUAD_BILATERAL_SWI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, U5 74LVC4066D_QUAD_BILATERAL_SWI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, U6 OPA344, U7 74LVC541A, U8 U-BLOX_ZED-F9P, U9 FIN1017MX

Commit message: Update post Reds review.
Line up USB Shield JP with CC resistors.
Relabel C8 with value, remove tolerance
Remove cap placement note.
Make USB Shield JP NC
Rename JPs to their function
Add USBSHLD Jumper text
Acid Traps
Label PPS header
Add measures
Align RST/EXTINT PTH in 0.1" grid
Move C3 back a bit from VREG
Move GND PTH back from C7
Relabel GRF as GND in silk
Recenter EXTINT AND RESET GND silk
Parts:
- removed JP3: JUMPER-SMT_2_NO_SILK, SparkFun-Jumpers:JUMPER-SMT_2_NO_SILK
- added USBSHLD: JUMPER-SMT_2_NC_TRACE_SILK, SparkFun-Jumpers:JUMPER-SMT_2_NC_TRACE_SILK
- C8: CAPACITANCE (none) -> 47pF
- R6, R8: value 1k -> 4.7k; device SparkFun-Resistors:1KOHM-0402T-1/16W-1% -> SparkFun-Resistors:4.7KOHM-0402T-1/16W-1%
- renumbered JP1 to USBPWR, JP2 to WP, JP4 to PWRLED, JP5 to RTKLED, JP6 to PPSLED, JP7 to I2CPUR, JP8 to ANTSUP, JP9 to DSEL
Connections:
- net GND: now also USBSHLD.2; no longer JP3.2
- net SHLD: now also USBSHLD.1; no longer JP3.1
Other:
- note added: "USBSHLD Jumper Use this jumper to connect/disconnect your USB-C cable shield to this PCB's GND. Closed (default): connected to GND"
- note removed: "1k"
- note removed: "Place capacitor as close as possible to module."
- note removed: "Place diode close to connector."
- moved on the sheet: D3, R10, R3, R4, R9

Commit message: Rev to v10.
Other:
- note added: "v10"
- note removed: "v03"
Changed lines of the file:
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@@
 <text x="71.374" y="86.106" size="2.54" layer="94" font="vector" align="center">MicroMod Function Connector</text>
 <text x="348.234" y="11.176" size="2.54" layer="94" font="vector">A. Brudner</text>
-<text x="421.894" y="6.096" size="2.54" layer="94" font="vector">v03</text>
+<text x="421.894" y="6.096" size="2.54" layer="94" font="vector">v10</text>
 <text x="71.12" y="269.24" size="2.54" layer="94" font="vector" align="center">ZED-F9P USB (u-center)</text>
 <text x="111.76" y="203.2" size="2.54" layer="94" font="vector" align="center">ZED-F9P Backup Battery</text>

Commit message: Retune LED brightness.
Per experiment Pete performed.

Red LED = 1kOhm @3.3V
Blue LED = 4.7kOhm @3.3V

Replaced Yellow LED with Blue LED to match design standards.
Parts:
- D6: value YELLOW -> BLUE; device SparkFun-LED:LED-YELLOW0603 -> SparkFun-LED:LED-BLUE0603
- R6: value 4.7k -> 1k; device SparkFun-Resistors:4.7KOHM-0402T-1/16W-1% -> SparkFun-Resistors:1KOHM-0402T-1/16W-1%
- R7: value 1k -> 4.7k; device SparkFun-Resistors:1KOHM-0402T-1/16W-1% -> SparkFun-Resistors:4.7KOHM-0402T-1/16W-1%
Changed lines of the file:
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@@
 <part name="SUPPLY20" library="SparkFun-PowerSymbols" deviceset="V_BATT" device=""/>
 <part name="SUPPLY21" library="SparkFun-PowerSymbols" deviceset="3.3V" device=""/>
-<part name="R7" library="SparkFun-Resistors" deviceset="1KOHM" device="-0402T-1/16W-1%" value="1k"/>
+<part name="R7" library="SparkFun-Resistors" deviceset="4.7KOHM" device="-0402T-1/16W-1%" value="4.7k"/>
 <part name="RTKLED" library="SparkFun-Jumpers" deviceset="JUMPER-SMT_2_NC_TRACE" device="_SILK" package3d_urn="urn:adsk.eagle:package:39281/1" value="JUMPER-SMT_2_NC_TRACE_SILK"/>
 <part name="D7" library="SparkFun-DiscreteSemi" deviceset="DIODE-SCHOTTKY" device="-PMEG4005EJ" value="0.5A/40V/420mV"/>
@@
 <part name="GND45" library="SparkFun-PowerSymbols" deviceset="GND" device=""/>
 <part name="GND46" library="SparkFun-PowerSymbols" deviceset="GND" device=""/>
-<part name="R6" library="SparkFun-Resistors" deviceset="4.7KOHM" device="-0402T-1/16W-1%" value="4.7k"/>
+<part name="R6" library="SparkFun-Resistors" deviceset="1KOHM" device="-0402T-1/16W-1%" value="1k"/>
 <part name="R20" library="SparkFun-Resistors" deviceset="10KOHM" device="-0402T-1/16W-1%" value="10k"/>
 <part name="SUPPLY11" library="SparkFun-PowerSymbols" deviceset="VDD" device="" value="V_ZED"/>
@@
 <part name="R8" library="SparkFun-Resistors" deviceset="4.7KOHM" device="-0402T-1/16W-1%" value="4.7k"/>
 <part name="PPSLED" library="SparkFun-Jumpers" deviceset="JUMPER-SMT_2_NC_TRACE" device="_SILK" package3d_urn="urn:adsk.eagle:package:39281/1" value="JUMPER-SMT_2_NC_TRACE_SILK"/>
-<part name="D6" library="SparkFun-LED" deviceset="LED-YELLOW" device="0603" value="YELLOW"/>
+<part name="D6" library="SparkFun-LED" deviceset="LED-BLUE" device="0603" value="BLUE"/>
 <part name="R11" library="SparkFun-Resistors" deviceset="2.2KOHM" device="-0402T-1/16W-1%" value="2.2k"/>
 <part name="R12" library="SparkFun-Resistors" deviceset="2.2KOHM" device="-0402T-1/16W-1%" value="2.2k"/>

Commit message: Decrease V_USB vdiv resistors.
Decrease by 2 orders of magnitude to allow more current flow for V_DETECT.
22k -> 220
47k -> 470
Parts:
- R18: value 22k -> 220; device SparkFun-Resistors:22KOHM-0402_TIGHT-1/10W-1% -> SparkFun-Resistors:220OHM-0402-TIGHT-1/16W-1%
- R19: value 47k -> 470; device SparkFun-Resistors:47KOHM-0402-1/10W-1% -> SparkFun-Resistors:470OHM-0402-TIGHT-1/16W-1%
Changed lines of the file:
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@@
 <part name="SUPPLY7" library="SparkFun-PowerSymbols" deviceset="V_BATT" device=""/>
 <part name="SUPPLY19" library="SparkFun-PowerSymbols" deviceset="VDD" device="" value="V_ZED"/>
-<part name="R19" library="SparkFun-Resistors" deviceset="47KOHM" device="-0402-1/10W-1%" value="47k"/>
+<part name="R19" library="SparkFun-Resistors" deviceset="470OHM" device="-0402-TIGHT-1/16W-1%" value="470"/>
 <part name="U8" library="SparkFun_MicroMod_GNSS_Function_Board_ZED-F9P" deviceset="U-BLOX_ZED-F9P" device=""/>
 <part name="C10" library="SparkFun-Capacitors" deviceset="0.1UF" device="-0402T-16V-10%" value="0.1uF"/>
@@
 <part name="GND33" library="SparkFun-PowerSymbols" deviceset="GND" device=""/>
 <part name="GND34" library="SparkFun-PowerSymbols" deviceset="GND" device=""/>
-<part name="R18" library="SparkFun-Resistors" deviceset="22KOHM" device="-0402_TIGHT-1/10W-1%" value="22k"/>
+<part name="R18" library="SparkFun-Resistors" deviceset="220OHM" device="-0402-TIGHT-1/16W-1%" value="220"/>
 <part name="J1" library="SparkFun-Connectors" deviceset="USB_C" device="_4-LAYER-ISOLATED" value="USB Female Type C Connector"/>
 <part name="J3" library="SparkFun-Connectors" deviceset="CONN_01" device="PTH_NO_SILK_YES_STOP"/>
