File: Hardware/SparkFun_MicroMod_GNSS_Function_Board_ZED-F9P.brd (EAGLE design)
At the start: 37.5 x 65 mm, 164 parts, among them J1 USB Female Type C Connector, J10 455-1750-1-ND, J2 MICROMOD_FUNCTION_STANDARD, J9 U.FL, Q1 DMP21D0UT-7, U1 NLAST4501DFT2G, U10 SN74AUP1T04, U11 SN74AUP1T04, U2 3.3V, U3 EEPROM, U4 74LVC4066D_QUAD_BILATERAL_SWI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, U5 74LVC4066D_QUAD_BILATERAL_SWI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, U6 OPA344, U7 74LVC541A, U8 U-BLOX_ZED-F9P, U9 FIN1017MX

Commit message: Rev to v10.
Other:
- board text added: "v10"
- board text removed: "v03"
Changed lines of the file:
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@@
 <plain>
 <wire x1="28.672" y1="0" x2="21.972" y2="0" width="0.05" layer="20"/>
-<text x="31.67" y="5.17" size="1.27" layer="16" font="vector" ratio="20" rot="SMR0" align="center">v03</text>
+<text x="31.67" y="5.17" size="1.27" layer="16" font="vector" ratio="20" rot="SMR0" align="center">v10</text>
 <text x="62.23" y="-8.89" size="1.778" layer="51" font="vector">A. Brudner</text>
 <wire x1="20.772" y1="0" x2="8.822" y2="0" width="0.05" layer="20"/>

Commit message: Retune LED brightness.
Per experiment Pete performed.

Red LED = 1kOhm @3.3V
Blue LED = 4.7kOhm @3.3V

Replaced Yellow LED with Blue LED to match design standards.
Parts:
- D6: value YELLOW -> BLUE
- R6: value 4.7k -> 1k
- R7: value 1k -> 4.7k
Changed lines of the file:
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@@
 <drawing>
 <settings>
-<setting alwaysvectorfont="yes"/>
+<setting alwaysvectorfont="no"/>
 <setting verticaltext="up"/>
 </settings>
@@
 <attribute name="RES" value="3.3k" x="18.99" y="9.51" size="1.778" layer="27" display="off"/>
 </element>
-<element name="R7" library="SparkFun-Resistors" package="0402-TIGHT" value="1k" x="8.5" y="61.35" smashed="yes" rot="R270">
+<element name="R7" library="SparkFun-Resistors" package="0402-TIGHT" value="4.7k" x="8.5" y="61.35" smashed="yes" rot="R270">
 <attribute name="NAME" x="8.262" y="59.15" size="0.6096" layer="25" font="vector" ratio="20" rot="R270" align="bottom-center"/>
-<attribute name="PROD_ID" value="RES-14342" x="13.5" y="87.35" size="1.778" layer="27" rot="R270" display="off"/>
-<attribute name="VALUE" value="1k" x="8.5" y="61.35" size="1.778" layer="27" rot="R270" display="off"/>
+<attribute name="PROD_ID" value="RES-15343" x="13.5" y="87.35" size="1.778" layer="27" rot="R270" display="off"/>
+<attribute name="VALUE" value="4.7k" x="8.5" y="61.35" size="1.778" layer="27" rot="R270" display="off"/>
 </element>
 <element name="RTKLED" library="SparkFun-Jumpers" package="SMT-JUMPER_2_NC_TRACE_SILK" package3d_urn="urn:adsk.eagle:package:39281/1" value="JUMPER-SMT_2_NC_TRACE_SILK" x="6.5" y="61.8" smashed="yes" rot="MR90">
@@
 <element name="U$73" library="output" package="#_DIS#0" value="" x="10.8" y="53.4" smashed="yes" rot="MR0"/>
 <element name="U$74" library="output" package="#EN_#0" value="" x="17.1" y="53.4" smashed="yes" rot="MR0"/>
-<element name="R6" library="SparkFun-Resistors" package="0402-TIGHT" value="4.7k" x="12.5" y="61.35" smashed="yes" rot="R270">
+<element name="R6" library="SparkFun-Resistors" package="0402-TIGHT" value="1k" x="12.5" y="61.35" smashed="yes" rot="R270">
 <attribute name="NAME" x="13.262" y="61.35" size="0.6096" layer="25" font="vector" ratio="20" rot="R270" align="bottom-center"/>
-<attribute name="PROD_ID" value="RES-15343" x="12.5" y="65.25" size="1.778" layer="27" rot="R270" display="off"/>
-<attribute name="VALUE" value="4.7k" x="11.738" y="61.35" size="0.6096" layer="27" font="vector" ratio="20" rot="R270" align="top-center"/>
+<attribute name="PROD_ID" value="RES-14342" x="12.5" y="65.25" size="1.778" layer="27" rot="R270" display="off"/>
+<attribute name="VALUE" value="1k" x="11.738" y="61.35" size="0.6096" layer="27" font="vector" ratio="20" rot="R270" align="top-center"/>
 </element>
 <element name="R20" library="SparkFun-Resistors" package="0402-TIGHT" value="10k" x="33.2" y="25.6" smashed="yes" rot="R90">
@@
 <attribute name="VALUE" x="1.357" y="61.8" size="0.6096" layer="28" font="vector" ratio="20" rot="MR90" align="top-center"/>
 </element>
-<element name="D6" library="SparkFun-LED" package="LED-0603" value="YELLOW" x="2.5" y="61.7" smashed="yes" rot="R270">
+<element name="D6" library="SparkFun-LED" package="LED-0603" value="BLUE" x="2.5" y="61.7" smashed="yes" rot="R270">
 <attribute name="NAME" x="3.135" y="61.7" size="0.6096" layer="25" font="vector" ratio="20" rot="R270" align="bottom-center"/>
-<attribute name="PROD_ID" value="DIO-09003" x="6.6" y="74.2" size="1.778" layer="27" rot="R270" display="off"/>
-<attribute name="VALUE" x="1.865" y="61.7" size="0.6096" layer="27" font="vector" ratio="20" rot="R270" align="top-center"/>
+<attribute name="PROD_ID" value="DIO-08575" x="6.6" y="74.2" size="1.778" layer="27" rot="R270" display="off"/>
+<attribute name="VALUE" value="BLUE" x="1.865" y="61.7" size="0.6096" layer="27" font="vector" ratio="20" rot="R270" align="top-center"/>
 </element>
 <element name="U$2" library="output" package="#_RTCMTX#0" value="" x="36" y="10.05" smashed="yes" rot="MR0"/>

Commit message: Decrease V_USB vdiv resistors.
Decrease by 2 orders of magnitude to allow more current flow for V_DETECT.
22k -> 220
47k -> 470
Parts:
- R18: value 22k -> 220
- R19: value 47k -> 470
Changed lines of the file:
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@@
 <attribute name="PROD_ID" value="DIO-00819" x="10.5" y="75.7" size="1.778" layer="27" rot="R270" display="off"/>
 </element>
-<element name="R19" library="SparkFun-Resistors" package="0402-TIGHT" value="47k" x="20.2" y="31" smashed="yes" rot="R90">
+<element name="R19" library="SparkFun-Resistors" package="0402-TIGHT" value="470" x="20.2" y="31" smashed="yes" rot="R90">
 <attribute name="NAME" x="19.538" y="31" size="0.6096" layer="25" font="vector" ratio="20" rot="R90" align="bottom-center"/>
-<attribute name="PROD_ID" value="RES-15011" x="0.2" y="27" size="1.778" layer="27" rot="R90" display="off"/>
-<attribute name="VALUE" value="47k" x="20.862" y="31" size="0.6096" layer="27" font="vector" ratio="20" rot="R90" align="top-center"/>
+<attribute name="PROD_ID" value="RES-15584" x="0.2" y="27" size="1.778" layer="27" rot="R90" display="off"/>
+<attribute name="VALUE" value="470" x="20.862" y="31" size="0.6096" layer="27" font="vector" ratio="20" rot="R90" align="top-center"/>
 </element>
 <element name="U8" library="SparkFun_MicroMod_GNSS_Function_Board_ZED-F9P" package="ZED-F9P" value="U-BLOX_ZED-F9P" x="15" y="43.3" smashed="yes" rot="R180">
@@
 <attribute name="VALUE" value="NLAST4501DFT2G" x="26.4" y="31.3" size="1.778" layer="27" rot="R270" display="off"/>
 </element>
-<element name="R18" library="SparkFun-Resistors" package="0402-TIGHT" value="22k" x="22.8" y="31.3" smashed="yes" rot="R180">
+<element name="R18" library="SparkFun-Resistors" package="0402-TIGHT" value="220" x="22.8" y="31.3" smashed="yes" rot="R180">
 <attribute name="NAME" x="22.8" y="30.062" size="0.6096" layer="25" font="vector" ratio="20" align="bottom-center"/>
-<attribute name="PROD_ID" value="RES-14281" x="22.8" y="31.3" size="1.778" layer="27" rot="R180" display="off"/>
-<attribute name="VALUE" value="22k" x="22.8" y="31.962" size="0.6096" layer="27" font="vector" ratio="20" rot="R180" align="top-center"/>
+<attribute name="PROD_ID" value="RES-15269" x="22.8" y="31.3" size="1.778" layer="27" rot="R180" display="off"/>
+<attribute name="VALUE" value="220" x="22.8" y="31.962" size="0.6096" layer="27" font="vector" ratio="20" rot="R180" align="top-center"/>
 </element>
 <element name="J1" library="SparkFun-Connectors" package="USB-C-16P-4LAYER-ISOLATED" value="USB Female Type C Connector" x="30.4" y="58.9" smashed="yes" rot="R180">
